Commit message: state_estimation using imu+odom implemented

File: gazebo/urdf/iBot.urdf (robot description, URDF)
Before this commit: robot iBot, 8 links, 7 joints
Links:
- link back_left_wheel: geometry collision cylinder length=0.05 radius=0.125; visual mesh filename=package://iBot/meshes/wheel.obj
- link back_right_wheel: geometry collision cylinder length=0.05 radius=0.125; visual mesh filename=package://iBot/meshes/wheel.obj
- link chassis: geometry collision box size=.4 .2 .1; visual mesh filename=package://iBot/meshes/chassis.obj
- link front_left_wheel: geometry collision cylinder length=0.05 radius=0.125; visual mesh filename=package://iBot/meshes/wheel.obj
- link front_right_wheel: geometry collision cylinder length=0.05 radius=0.125; visual mesh filename=package://iBot/meshes/wheel.obj

File: gazebo/urdf/iBot.urdf.xacro (robot description, xacro)
@@ -23,8 +23,10 @@
     </collision>
     <visual name='chassis_visual'>
-      <origin xyz="0 0 0" rpy=" 0 0 0"/>
-      <geometry>
-        <box size=".4 .2 .1"/>
-      </geometry>
+      <origin xyz="0 -0.1 0" rpy=" 0 0 0"/>
+      <geometry>
+        <mesh filename="package://iBot/meshes/chassis.obj"/>
+      </geometry>
+      <transparency>0</transparency>
+      <cast_shadows>1</cast_shadows>
     </visual>
   </link>
@@ -33,49 +35,55 @@
       <mass value="5.0"/>
       <origin xyz="0.0 0 0" rpy=" 0 1.5707 1.5707"/>
+      <inertia ixx="0.0285" ixy="0" ixz="0" iyy="0.0285" iyz="0" izz="0.0391" />
+    </inertial>
+    <visual>
+      <origin xyz="0 -0.025 0" rpy=" 0 0 0"/>
+      <geometry>
+        <mesh filename="package://iBot/meshes/wheel.obj"/>
+      </geometry>
+      <transparency>0</transparency>
+      <cast_shadows>1</cast_shadows>
+    </visual>
+    <collision>
+      <origin xyz="0.0 0 0" rpy=" 0 1.5707 1.5707"/>
+      <geometry>
+        <cylinder length="0.05" radius="0.125"/>
+      </geometry>
+    </collision>
+  </link>
+  <link name="back_left_wheel">
+    <inertial>
+      <mass value="5.0"/>
+      <origin xyz="0.0 0 0" rpy=" 0 1.5707 1.5707"/>
+      <inertia ixx="0.0285" ixy="0" ixz="0" iyy="0.0285" iyz="0" izz="0.0391" />
+    </inertial>
+    <visual>
+      <origin xyz="0 -0.025 0" rpy=" 0 0 0"/>
+      <geometry>
+        <mesh filename="package://iBot/meshes/wheel.obj"/>
+      </geometry>
+      <transparency>0</transparency>
+      <cast_shadows>1</cast_shadows>
+    </visual>
+    <collision>
+      <origin xyz="0.0 0 0" rpy=" 0 1.5707 1.5707"/>
+      <geometry>
+        <cylinder length="0.05" radius="0.125"/>
+      </geometry>
+    </collision>
+  </link>
+  <link name="front_right_wheel">
+    <inertial>
+      <mass value="5.0"/>
+      <origin xyz="0.0 0 0" rpy=" 0 1.5707 1.5707"/>
       <inertia ixx="0.1" ixy="0" ixz="0" iyy="0.1" iyz="0" izz="0.1" />
     </inertial>
     <visual>
-      <origin xyz="0.0 0 0" rpy=" 0 1.5707 1.5707"/>
-      <geometry>
-        <cylinder length="0.05" radius="0.125"/>
-      </geometry>
-    </visual>
-    <collision>
-      <origin xyz="0.0 0 0" rpy=" 0 1.5707 1.5707"/>
-      <geometry>
-        <cylinder length="0.05" radius="0.125"/>
-      </geometry>
-    </collision>
-  </link>
-  <link name="back_left_wheel">
-    <inertial>
-      <mass value="5.0"/>
-      <origin xyz="0.0 0 0" rpy=" 0 1.5707 1.5707"/>
-      <inertia ixx="0.1" ixy="0" ixz="0" iyy="0.1" iyz="0" izz="0.1" />
-    </inertial>
-    <visual>
-      <origin xyz="0.0 0 0" rpy=" 0 1.5707 1.5707"/>
-      <geometry>
-        <cylinder length="0.05" radius="0.125"/>
-      </geometry>
-    </visual>
-    <collision>
-      <origin xyz="0.0 0 0" rpy=" 0 1.5707 1.5707"/>
-      <geometry>
-        <cylinder length="0.05" radius="0.125"/>
-      </geometry>
-    </collision>
-  </link>
-  <link name="front_right_wheel">
-    <inertial>
-      <mass value="5.0"/>
-      <origin xyz="0.0 0 0" rpy=" 0 1.5707 1.5707"/>
-      <inertia ixx="0.1" ixy="0" ixz="0" iyy="0.1" iyz="0" izz="0.1" />
-    </inertial>
-    <visual>
-      <origin xyz="0.0 0 0" rpy=" 0 1.5707 1.5707"/>
-      <geometry>
-        <cylinder length="0.05" radius="0.125"/>
-      </geometry>
+      <origin xyz="0 -0.025 0" rpy=" 0 0 0"/>
+      <geometry>
+        <mesh filename="package://iBot/meshes/wheel.obj"/>
+      </geometry>
+      <transparency>0</transparency>
+      <cast_shadows>1</cast_shadows>
     </visual>
     <collision>
@@ -90,11 +98,13 @@
       <mass value="5.0"/>
       <origin xyz="0.0 0 0" rpy=" 0 1.5707 1.5707"/>
-      <inertia ixx="0.1" ixy="0" ixz="0" iyy="0.1" iyz="0" izz="0.1" />
-    </inertial>
-    <visual>
-      <origin xyz="0.0 0 0" rpy=" 0 1.5707 1.5707"/>
-      <geometry>
-        <cylinder length="0.05" radius="0.125"/>
-      </geometry>
+      <inertia ixx="0.0285" ixy="0" ixz="0" iyy="0.0285" iyz="0" izz="0.0391" />
+    </inertial>
+    <visual>
+      <origin xyz="0 -0.025 0" rpy=" 0 0 0"/>
+      <geometry>
+        <mesh filename="package://iBot/meshes/wheel.obj"/>
+      </geometry>
+      <transparency>0</transparency>
+      <cast_shadows>1</cast_shadows>
     </visual>
     <collision>
@@ -185,9 +195,9 @@
     <parent link="chassis"/>
   </joint>
-  <gazebo reference="chassis">
+  <!-- <gazebo reference="chassis">
     <material>Gazebo/Blue</material>
-  </gazebo>
+  </gazebo> -->
   <gazebo reference="camera">
-    <material>Gazebo/Red</material>
+    <material>Gazebo/Blue</material>
   </gazebo>
   <gazebo reference="imu">
