Commit message: README updated

File: gazebo/models/iBot/iBot.urdf (robot description, URDF)
Before this commit: robot iBot, 8 links, 7 joints
Links:
- added link camera_frame
Joints:
- added joint camera_frame_joint: type fixed, parent camera, child camera_frame, origin xyz=0.025 0 0 rpy=-1.5707963267948966 0 -1.5707963267948966

File: gazebo/models/iBot/iBot.urdf.xacro (robot description, xacro)
@@ -133,4 +133,10 @@
     <child link="camera"/>
   </joint>
+  <link name="camera_frame"/>
+  <joint name="camera_frame_joint" type="fixed">
+    <origin xyz="${camera_length/2} 0 0" rpy="${-pi/2} 0 ${-pi/2}"/>
+    <parent link="camera"/>
+    <child link="camera_frame"/>
+  </joint>
   <!-- ************************** IMU *************************** -->
   <link name="imu">
