Commit message: navigation pkg initial commit. add caster wheel to bot.

File: simulation/models/iBot/iBot.urdf (robot description, URDF)
Before this commit: robot iBot, 9 links, 8 joints
Links:
- removed link front_left_wheel_link
- removed link front_right_wheel_link
- added link caster_front_link, mass 5; collision sphere radius=0.04; visual sphere radius=0.04
Joints:
- removed joint front_left_wheel_joint
- removed joint front_right_wheel_joint
- added joint caster_front_joint: type revolute, parent chassis, child caster_front_link, origin xyz=0.115 0.0 -0.09 rpy=0 0 0, axis 0 1 0, limit lower=-1e+16 upper=1e+16 effort=1000 velocity=1000

Commit message: Fixed Trajectory Follower and URDF

File: simulation/models/iBot/iBot.urdf (robot description, URDF)
Before this commit: robot iBot, 8 links, 7 joints
Links:
- removed link caster_front_link
- added link front_left_wheel_link, mass 7; collision cylinder length=0.1 radius=0.125; visual mesh filename=package://iBot/meshes/wheel3.obj
- added link front_right_wheel_link, mass 7; collision cylinder length=0.1 radius=0.125; visual mesh filename=package://iBot/meshes/wheel3.obj
- link back_left_wheel_link: mass 5 -> 7
- link back_right_wheel_link: mass 5 -> 7
Joints:
- removed joint caster_front_joint
- added joint front_left_wheel_joint: type revolute, parent chassis, child front_left_wheel_link, origin xyz=0.175 0.16000000000000003 -0.025 rpy=0 0 0, axis 0 1 0, limit lower=-1e+16 upper=1e+16 effort=1000 velocity=1000
- added joint front_right_wheel_joint: type revolute, parent chassis, child front_right_wheel_link, origin xyz=0.175 -0.16000000000000003 -0.025 rpy=0 0 0, axis 0 1 0, limit lower=-1e+16 upper=1e+16 effort=1000 velocity=1000

File: simulation/models/iBot/iBot.urdf.xacro (robot description, xacro)
@@ -21,5 +21,6 @@
       <origin xyz="0 0 0" rpy="${pi/2} 0 0" />
       <mass value="${m}"/>
-      <inertia ixx="${(m/12) * (3*r*r + h*h)}" ixy = "0" ixz = "0" iyy="${(m/12) * (3*r*r + h*h)}" iyz = "0" izz="${(m/2) * (r*r)}"/>
+      <!-- <inertia ixx="${(m/12) * (3*r*r + h*h)}" ixy = "0" ixz = "0" iyy="${(m/12) * (3*r*r + h*h)}" iyz = "0" izz="${(m/2) * (r*r)}"/> -->
+      <inertia ixx="2.369791666666667" ixy="0" ixz="0" iyy="2.369791666666667" iyz="0" izz="3.90625" />
     </inertial>
   </xacro:macro>
@@ -28,5 +29,6 @@
       <origin xyz="0 0 0" rpy="${pi/2} 0 ${pi/2}"/>
       <mass value="${m}"/>
-      <inertia ixx="${(m/12) * (h*h + d*d)}" ixy="0.0" ixz="0.0" iyy="${(m/12) * (w*w + d*d)}" iyz="0.0" izz="${(m/12) * (w*w + h*h)}"/>
+      <!-- <inertia ixx="${(m/12) * (h*h + d*d)}" ixy="0.0" ixz="0.0" iyy="${(m/12) * (w*w + d*d)}" iyz="0.0" izz="${(m/12) * (w*w + h*h)}"/> -->
+      <inertia ixx="0.21250000000000005" ixy="0.0" ixz="0.0" iyy="0.25000000000000006" iyz="0.0" izz="0.06250000000000001" />
     </inertial>
   </xacro:macro>
@@ -83,11 +85,11 @@
         <friction>
           <ode>
-            <mu>500</mu>
-            <mu2>500</mu2>
+            <mu>10.0</mu>
+            <mu2>5.0</mu2>
           </ode>
         </friction>
       </surface>
       </collision>
-      <xacro:cylinder_inertia m="5" r="${wheel_radius}" h="${wheel_width}"/>
+      <xacro:cylinder_inertia m="7" r="${wheel_radius}" h="${wheel_width}"/>
     </link>
     <joint name="${prefix}_joint" type="revolute">
